Commit message: First commit of Groovy development branch

File: branches/groovy/rbx_vol_1/rbx1_description/urdf/turtlebot.xacro (robot description, xacro)
@@ -2,5 +2,5 @@
 <robot>
   <include filename="$(find rbx1_description)/urdf/turtlebot_hardware.xacro" />
-  <include filename="$(find turtlebot_description)/urdf/gazebo.urdf.xacro"/>
+  <include filename="$(find rbx1_description)/urdf/gazebo.urdf.xacro"/>
   <material name="Green">
     <color rgba="0.0 0.8 0.0 1.0"/>
@@ -47,5 +47,5 @@
       <origin xyz=" 0 0 0.0308" rpy="0 0 0" />
       <geometry>
-        <mesh filename="package://turtlebot_description/meshes/create_body.dae" />
+        <mesh filename="package://rbx1_description/meshes/create_body.dae" />
       </geometry>
     </visual>
@@ -291,5 +291,5 @@
       <origin xyz=" 0 0 0 " rpy="0 0 0" />
       <geometry>
-        <mesh filename="package://turtlebot_description/meshes/plate_0_logo.dae"/>
+        <mesh filename="package://rbx1_description/meshes/plate_0_logo.dae"/>
       </geometry>
     </visual>
@@ -321,5 +321,5 @@
       <origin xyz=" 0 0 0 " rpy="0 0 0" />
       <geometry>
-        <mesh filename="package://turtlebot_description/meshes/plate_1_logo.dae"/>
+        <mesh filename="package://rbx1_description/meshes/plate_1_logo.dae"/>
       </geometry>
     </visual>
@@ -351,5 +351,5 @@
       <origin xyz=" 0 0 0 " rpy="0 0 0" />
       <geometry>
-        <mesh filename="package://turtlebot_description/meshes/plate_1_logo.dae"/>
+        <mesh filename="package://rbx1_description/meshes/plate_1_logo.dae"/>
       </geometry>
     </visual>
@@ -474,5 +474,5 @@
       <origin xyz=" 0 0 0 " rpy="0 0 0" />
       <geometry>
-        <mesh filename="package://turtlebot_description/meshes/plate_2_logo.dae"/>
+        <mesh filename="package://rbx1_description/meshes/plate_2_logo.dae"/>
       </geometry>
     </visual>
